Commit message: Fixing and editing the physics

File: src/physics/src/model.urdf (robot description, URDF)
Before this commit: robot edo_sim, 7 links, 6 joints
Links:
- link base_link: geometry collision mesh filename=/home/khush_24_01/Robo_arm_ctrl/install/meshes/share/meshes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; visual mesh filename=/home/khush_24_01/Robo_arm_ctrl/install/meshes/share/meshes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
- link link_1: geometry collision mesh filename=/home/khush_24_01/Robo_arm_ctrl/install/meshes/share/meshes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; visual mesh filename=/home/khush_24_01/Robo_arm_ctrl/install/meshes/share/meshes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
- link link_2: geometry collision mesh filename=/home/khush_24_01/Robo_arm_ctrl/install/meshes/share/meshes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; visual mesh filename=/home/khush_24_01/Robo_arm_ctrl/install/meshes/share/meshes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
- link link_3: geometry collision mesh filename=/home/khush_24_01/Robo_arm_ctrl/install/meshes/share/meshes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; visual mesh filename=/home/khush_24_01/Robo_arm_ctrl/install/meshes/share/meshes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
- link link_4: geometry collision mesh filename=/home/khush_24_01/Robo_arm_ctrl/install/meshes/share/meshes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; visual mesh filename=/home/khush_24_01/Robo_arm_ctrl/install/meshes/share/meshes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
- link link_5: geometry collision mesh filename=/home/khush_24_01/Robo_arm_ctrl/install/meshes/share/meshes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; visual mesh filename=/home/khush_24_01/Robo_arm_ctrl/install/meshes/share/meshes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
- link link_6: geometry collision mesh filename=/home/khush_24_01/Robo_arm_ctrl/install/meshes/share/meshes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; visual mesh filename=/home/khush_24_01/Robo_arm_ctrl/install/meshes/share/meshes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
